File: device.sch (EAGLE design)
At the start: 33 parts, among them P1 ST9S008V4AR1500, P2 S2B-PH-SM4-TB(LF)(SN), Q1 FDN340P, U1 RPI_COMPUTE, U2 LMR10510YMFE/NOPB, U3 LMR10510YMFE/NOPB, U4 MCP73832T-2ACI/OT

Commit message: Add Wi-Fi
Parts:
- added R15, R16, R17, R18, R19, R20: 33, resistor:R-EU_R0603
- added U5: (no value), esp8266modules:ESP12ESMD
Connections:
- new net N$15: R15.2, U5.SCLK
- new net N$16: R16.2, U5.MOSI
- new net N$17: R17.2, U5.*GPIO10
- new net N$18: R18.2, U5.*GPIO9
- new net N$19: R19.2, U5.MISO
- new net N$20: R20.2, U5.CS0
- new net SDIO_CLK: R15.1, U1.75/GPIO22
- new net SDIO_CMD: R20.1, U1.77/GPIO23
- new net SDIO_D0: R19.1, U1.81/GPIO24
- new net SDIO_D1: R16.1, U1.83/GPIO25
- new net SDIO_D2: R18.1, U1.87/GPIO26
- new net SDIO_D3: R17.1, U1.89/GPIO27
- new net SDIO_ID: U1.3/GPIO0, U5.CH_PD
- net +CM_3V3: now also U5.VCC
- net GND: now also U5.GND
Changed lines of the file:
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@@
 <part name="GND11" library="supply1" library_urn="urn:adsk.eagle:library:371" deviceset="GND" device=""/>
 <part name="GND13" library="supply1" library_urn="urn:adsk.eagle:library:371" deviceset="GND" device=""/>
+<part name="U5" library="esp8266modules" deviceset="ESP12E" device="SMD"/>
+<part name="GND14" library="supply1" library_urn="urn:adsk.eagle:library:371" deviceset="GND" device=""/>
+<part name="R15" library="resistor" library_urn="urn:adsk.eagle:library:348" deviceset="R-EU_" device="R0603" value="33"/>
+<part name="R16" library="resistor" library_urn="urn:adsk.eagle:library:348" deviceset="R-EU_" device="R0603" value="33"/>
+<part name="R17" library="resistor" library_urn="urn:adsk.eagle:library:348" deviceset="R-EU_" device="R0603" value="33"/>
+<part name="R18" library="resistor" library_urn="urn:adsk.eagle:library:348" deviceset="R-EU_" device="R0603" value="33"/>
+<part name="R19" library="resistor" library_urn="urn:adsk.eagle:library:348" deviceset="R-EU_" device="R0603" value="33"/>
+<part name="R20" library="resistor" library_urn="urn:adsk.eagle:library:348" deviceset="R-EU_" device="R0603" value="33"/>
 </parts>
 <sheets>
@@
 <instance part="GND11" gate="1" x="312.42" y="365.76"/>
 <instance part="GND13" gate="1" x="261.62" y="365.76"/>
+<instance part="U5" gate="G$1" x="449.58" y="195.58"/>
+<instance part="GND14" gate="1" x="469.9" y="167.64"/>
+<instance part="R15" gate="G$1" x="457.2" y="147.32" rot="R90"/>
+<instance part="R16" gate="G$1" x="449.58" y="147.32" rot="R90"/>
+<instance part="R17" gate="G$1" x="441.96" y="147.32" rot="R90"/>
+<instance part="R18" gate="G$1" x="434.34" y="147.32" rot="R90"/>
+<instance part="R19" gate="G$1" x="426.72" y="147.32" rot="R90"/>
+<instance part="R20" gate="G$1" x="419.1" y="147.32" rot="R90"/>
 </instances>
 <busses>
@@
 <wire x1="320.04" y1="297.18" x2="335.28" y2="297.18" width="0.762" layer="92"/>
 <label x="322.58" y="294.64" size="1.778" layer="95"/>
+</segment>
+</bus>
+<bus name="SDIO_D[0..3]">
+<segment>
+<wire x1="154.94" y1="200.66" x2="154.94" y2="213.36" width="0.762" layer="92"/>
+<wire x1="154.94" y1="213.36" x2="142.24" y2="213.36" width="0.762" layer="92"/>
+<label x="139.7" y="210.82" size="1.778" layer="95"/>
+</segment>
+<segment>
+<wire x1="391.16" y1="127" x2="391.16" y2="147.32" width="0.762" layer="92"/>
+<wire x1="391.16" y1="127" x2="449.58" y2="127" width="0.762" layer="92"/>
+<label x="386.08" y="149.86" size="1.778" layer="95"/>
 </segment>
 </bus>
@@
 <junction x="312.42" y="370.84"/>
 </segment>
+<segment>
+<pinref part="U5" gate="G$1" pin="GND"/>
+<pinref part="GND14" gate="1" pin="GND"/>
+<wire x1="464.82" y1="185.42" x2="469.9" y2="185.42" width="0.1524" layer="91"/>
+<wire x1="469.9" y1="185.42" x2="469.9" y2="170.18" width="0.1524" layer="91"/>
+</segment>
 </net>
 <net name="N$6" class="0">
@@
 <label x="292.1" y="492.76" size="1.778" layer="95"/>
 </segment>
+<segment>
+<pinref part="U5" gate="G$1" pin="VCC"/>
+<wire x1="431.8" y1="185.42" x2="421.64" y2="185.42" width="0.1524" layer="91"/>
+<label x="419.1" y="185.42" size="1.778" layer="95"/>
+</segment>
 </net>
 <net name="N$4" class="1">
@@
 </segment>
 </net>
+<net name="SDIO_ID" class="0">
+<segment>
+<pinref part="U1" gate="G$1" pin="3/GPIO0"/>
+<wire x1="182.88" y1="309.88" x2="160.02" y2="309.88" width="0.1524" layer="91"/>
+<label x="160.02" y="309.88" size="1.778" layer="95"/>
+</segment>
+<segment>
+<pinref part="U5" gate="G$1" pin="CH_PD"/>
+<wire x1="431.8" y1="198.12" x2="406.4" y2="198.12" width="0.1524" layer="91"/>
+<wire x1="406.4" y1="198.12" x2="406.4" y2="134.62" width="0.1524" layer="91"/>
+<label x="403.86" y="132.08" size="1.778" layer="95"/>
+</segment>
+</net>
+<net name="SDIO_CLK" class="0">
+<segment>
+<pinref part="U1" gate="G$1" pin="75/GPIO22"/>
+<wire x1="182.88" y1="218.44" x2="162.56" y2="218.44" width="0.1524" layer="91"/>
+<label x="162.56" y="218.44" size="1.778" layer="95"/>
+</segment>
+<segment>
+<pinref part="R15" gate="G$1" pin="1"/>
+<wire x1="457.2" y1="142.24" x2="457.2" y2="134.62" width="0.1524" layer="91"/>
+<label x="452.12" y="137.16" size="1.778" layer="95"/>
+</segment>
+</net>
+<net name="SDIO_CMD" class="0">
+<segment>
+<pinref part="U1" gate="G$1" pin="77/GPIO23"/>
+<wire x1="182.88" y1="215.9" x2="162.56" y2="215.9" width="0.1524" layer="91"/>
+<label x="162.56" y="215.9" size="1.778" layer="95"/>
+</segment>
+<segment>
+<pinref part="R20" gate="G$1" pin="1"/>
+<wire x1="419.1" y1="142.24" x2="419.1" y2="134.62" width="0.1524" layer="91"/>
+<label x="411.48" y="139.7" size="1.778" layer="95"/>
+</segment>
+</net>
+<net name="SDIO_D0" class="0">
+<segment>
+<pinref part="U1" gate="G$1" pin="81/GPIO24"/>
+<wire x1="182.88" y1="210.82" x2="154.94" y2="210.82" width="0.1524" layer="91"/>
+<label x="162.56" y="210.82" size="1.778" layer="95"/>
+</segment>
+<segment>
+<pinref part="R19" gate="G$1" pin="1"/>
+<label x="421.64" y="137.16" size="1.778" layer="95"/>
+<wire x1="426.72" y1="127" x2="426.72" y2="142.24" width="0.1524" layer="91"/>
+</segment>
+</net>
+<net name="SDIO_D1" class="0">
+<segment>
+<pinref part="U1" gate="G$1" pin="83/GPIO25"/>
+<wire x1="182.88" y1="208.28" x2="154.94" y2="208.28" width="0.1524" layer="91"/>
+<label x="162.56" y="208.28" size="1.778" layer="95"/>
+</segment>
+<segment>
+<pinref part="R16" gate="G$1" pin="1"/>
+<label x="444.5" y="139.7" size="1.778" layer="95"/>
+<wire x1="449.58" y1="127" x2="449.58" y2="142.24" width="0.1524" layer="91"/>
+</segment>
+</net>
+<net name="SDIO_D2" class="0">
+<segment>
+<pinref part="U1" gate="G$1" pin="87/GPIO26"/>
+<wire x1="182.88" y1="203.2" x2="154.94" y2="203.2" width="0.1524" layer="91"/>
+<label x="162.56" y="203.2" size="1.778" layer="95"/>
+</segment>
+<segment>
+<pinref part="R18" gate="G$1" pin="1"/>
+<label x="429.26" y="139.7" size="1.778" layer="95"/>
+<wire x1="434.34" y1="127" x2="434.34" y2="142.24" width="0.1524" layer="91"/>
+</segment>
+</net>
+<net name="SDIO_D3" class="0">
+<segment>
+<pinref part="U1" gate="G$1" pin="89/GPIO27"/>
+<wire x1="182.88" y1="200.66" x2="154.94" y2="200.66" width="0.1524" layer="91"/>
+<label x="162.56" y="200.66" size="1.778" layer="95"/>
+</segment>
+<segment>
+<pinref part="R17" gate="G$1" pin="1"/>
+<label x="436.88" y="137.16" size="1.778" layer="95"/>
+<wire x1="441.96" y1="127" x2="441.96" y2="142.24" width="0.1524" layer="91"/>
+</segment>
+</net>
+<net name="N$15" class="0">
+<segment>
+<pinref part="U5" gate="G$1" pin="SCLK"/>
+<wire x1="454.66" y1="167.64" x2="454.66" y2="154.94" width="0.1524" layer="91"/>
+<pinref part="R15" gate="G$1" pin="2"/>
+<wire x1="454.66" y1="154.94" x2="457.2" y2="154.94" width="0.1524" layer="91"/>
+<wire x1="457.2" y1="154.94" x2="457.2" y2="152.4" width="0.1524" layer="91"/>
+</segment>
+</net>
+<net name="N$16" class="0">
+<segment>
+<pinref part="U5" gate="G$1" pin="MOSI"/>
+<wire x1="452.12" y1="167.64" x2="452.12" y2="154.94" width="0.1524" layer="91"/>
+<pinref part="R16" gate="G$1" pin="2"/>
+<wire x1="452.12" y1="154.94" x2="449.58" y2="154.94" width="0.1524" layer="91"/>
+<wire x1="449.58" y1="154.94" x2="449.58" y2="152.4" width="0.1524" layer="91"/>
+</segment>
+</net>
+<net name="N$17" class="0">
+<segment>
+<pinref part="U5" gate="G$1" pin="*GPIO10"/>
+<wire x1="449.58" y1="167.64" x2="449.58" y2="157.48" width="0.1524" layer="91"/>
+<pinref part="R17" gate="G$1" pin="2"/>
+<wire x1="449.58" y1="157.48" x2="441.96" y2="157.48" width="0.1524" layer="91"/>
+<wire x1="441.96" y1="157.48" x2="441.96" y2="152.4" width="0.1524" layer="91"/>
+</segment>
+</net>
+<net name="N$18" class="0">
+<segment>
+<pinref part="U5" gate="G$1" pin="*GPIO9"/>
+<wire x1="447.04" y1="167.64" x2="447.04" y2="160.02" width="0.1524" layer="91"/>
+<pinref part="R18" gate="G$1" pin="2"/>
+<wire x1="447.04" y1="160.02" x2="434.34" y2="160.02" width="0.1524" layer="91"/>
+<wire x1="434.34" y1="160.02" x2="434.34" y2="152.4" width="0.1524" layer="91"/>
+</segment>
+</net>
+<net name="N$19" class="0">
+<segment>
+<pinref part="U5" gate="G$1" pin="MISO"/>
+<wire x1="444.5" y1="167.64" x2="444.5" y2="162.56" width="0.1524" layer="91"/>
+<pinref part="R19" gate="G$1" pin="2"/>
+<wire x1="444.5" y1="162.56" x2="426.72" y2="162.56" width="0.1524" layer="91"/>
+<wire x1="426.72" y1="162.56" x2="426.72" y2="152.4" width="0.1524" layer="91"/>
+</segment>
+</net>
+<net name="N$20" class="0">
+<segment>
+<pinref part="U5" gate="G$1" pin="CS0"/>
+<wire x1="441.96" y1="167.64" x2="441.96" y2="165.1" width="0.1524" layer="91"/>
+<pinref part="R20" gate="G$1" pin="2"/>
+<wire x1="441.96" y1="165.1" x2="419.1" y2="165.1" width="0.1524" layer="91"/>
+<wire x1="419.1" y1="165.1" x2="419.1" y2="152.4" width="0.1524" layer="91"/>
+</segment>
+</net>

Commit message: Modify layout and add PAM2306
Parts:
- removed CHARGE: (no value), led:LEDCHIP-LED0603
- removed D2, D3: (no value), diode:SCHOTTKY-DIODESMD
- removed R20: 33, resistor:R-EU_R0603
- removed U4: MCP73832T-2ACI/OT, Common-Parts-Library-Eagle:MCP73832T-2ACI/OT
- removed U5: (no value), esp8266modules:ESP12ESMD
- added C10, C5, C6, C7, C9: 10uF, resistor:C-EUC0603
- added C8: 100nF, resistor:C-EUC0603
- added LED2: (no value), led:LEDCHIP-LED0603
- added PCB1: RPI_COMPUTE, e14_Rpi_Compute_RevC:RPI_COMPUTE
- C1: value 22uF -> 10uF
- C2: value 22uF -> 1uF
- C3, C4: value 22uF -> 2.7uF
- J1: value (none) -> 10103594-0001LF; device Wurth_Elektronik_Electromechanic_Input-Output_Connectors_rev17b:632723100011 -> Common-Parts-Library-Eagle:10103594-0001LF
- L1, L2: value 1.6uH -> 4.7uH
- P1: value ST9S008V4AR1500 -> S2B-PH-SM4-TB(LF)(SN); device Common-Parts-Library-Eagle:ST9S008V4AR1500 -> Common-Parts-Library-Eagle:S2B-PH-SM4-TB(LF)(SN)
- P2: value S2B-PH-SM4-TB(LF)(SN) -> ST9S008V4AR1500; device Common-Parts-Library-Eagle:S2B-PH-SM4-TB(LF)(SN) -> Common-Parts-Library-Eagle:ST9S008V4AR1500
- Q1: value FDN340P -> SSM3J328R,LF; device Common-Parts-Library-Eagle:FDN340P -> Common-Parts-Library-Eagle:SSM3J328R,LF
- R1: value 45K -> 100K
- R11: value 470 -> 100K
- R12: value 2K -> 100K
- R14: value 470 -> 33
- R2: value 10K -> 470
- R3: value 100K -> 54K
- R4: value 20K -> 12K
- R5: value 10K -> 20K
- R7: value 100K -> 10K
- R8: value 100K -> 470
- R9: value 100K -> 2K
- U1: value RPI_COMPUTE -> PAM2306DYPAA; device e14_Rpi_Compute_RevC:RPI_COMPUTE -> PAM2306DYPAA:PAM2306DYPAA
- U2: value LMR10510YMFE/NOPB -> MCP73832T-2ACI/OT; device Common-Parts-Library-Eagle:LMR10510YMFE/NOPB -> Common-Parts-Library-Eagle:MCP73832T-2ACI/OT
- U3: value LMR10510YMFE/NOPB -> (none); device Common-Parts-Library-Eagle:LMR10510YMFE/NOPB -> esp8266modules:ESP12ESMD
- renumbered POWER to LED1
Connections:
- removed net N$13: R4.2, R5.2, U3.FB
- new net USB_OTGID: PCB1.168/USB_OTGID
- net +CM_1V8: now also C6.2, C7.2, PCB1.183/1V8, PCB1.184/1V8, PCB1.185/1V8, PCB1.186/1V8, R5.2; no longer C4.2, R4.1, U1.183/1V8, U1.184/1V8, U1.185/1V8, U1.186/1V8
- net +CM_3V3: now also C1.2, C5.2, P2.VCC, PCB1.189/VDAC, PCB1.190/VDAC, PCB1.191/3V3, PCB1.192/3V3, PCB1.193/3V3, PCB1.194/3V3, PCB1.197/VBAT, PCB1.198/VBAT, PCB1.199/VBAT, PCB1.200/VBAT, PCB1.39/GPIO0-27_VREF, PCB1.4/NC, PCB1.40/GPIO0-27_VREF, PCB1.41/GPIO28-45_VREF, PCB1.42/GPIO28-45_VREF, PCB1.6/NC, R2.2, R3.2, U3.VCC; no longer C2.2, P1.VCC, R1.1, R14.2, R6.2, U1.189/VDAC, U1.190/VDAC, U1.191/3V3, U1.192/3V3, U1.193/3V3, U1.194/3V3, U1.197/VBAT, U1.198/VBAT, U1.199/VBAT, U1.200/VBAT, U1.39/GPIO0-27_VREF, U1.4/NC, U1.40/GPIO0-27_VREF, U1.41/GPIO28-45_VREF, U1.42/GPIO28-45_VREF, U1.6/NC, U5.VCC
- net +VBAT: now also C3.2, P1.1, U2.VBAT; no longer P2.1, U4.VBAT
- net +VSUP: now also C4.2, D1.A, J1.VCC, R1.2, R8.2, U2.VDD; no longer D3.A, J1G$1.VBUS, J1G$1.VBUS1, J1G$1.VBUS2, J1G$1.VBUS3, R11.2, R13.2, U4.VDD
- net +VSYS: now also C10.2, C2.2, C9.2, D1.C, R6.2, U1.EN1, U1.VIN1, U1.VIN2; no longer C1.2, C3.2, D3.C, R3.2, U2.VIN, U3.VIN
- net GND: now also C10.1, C6.1, C8.1, C9.1, J1.GND, P1.2, P2.GND, PCB1.1/GND, PCB1.103/GND, PCB1.104/GND, PCB1.109/GND, PCB1.110/GND, PCB1.115/GND, PCB1.116/GND, PCB1.121/GND, PCB1.13/GND, PCB1.133/GND, PCB1.134/GND, PCB1.139/GND, PCB1.14/NC, PCB1.140/GND, PCB1.145/GND, PCB1.146/GND, PCB1.151/GND, PCB1.152/GND, PCB1.163/GND, PCB1.164/GND, PCB1.169/GND, PCB1.170/GND, PCB1.181/GND, PCB1.182/GND, PCB1.187/GND, PCB1.188/GND, PCB1.19/GND, PCB1.195/GND, PCB1.196/GND, PCB1.20/NC, PCB1.25/GND, PCB1.26/GND, PCB1.31/GND, PCB1.32/GND, PCB1.37/GND, PCB1.38/GND, PCB1.43/GND, PCB1.44/GND, PCB1.49/GND, PCB1.50/GND, PCB1.55/GND, PCB1.56/GND, PCB1.61/GND, PCB1.62/GND, PCB1.67/GND, PCB1.68/GND, PCB1.7/GND, PCB1.73/GND, PCB1.74/GND, PCB1.79/GND, PCB1.8/NC, PCB1.80/GND, PCB1.85/GND, PCB1.86/GND, PCB1.91/GND, PCB1.92/GND, PCB1.97/GND, PCB1.98/GND, R1.1, R11.1, R4.1, U1.EXP, U1.GND@1, U1.GND@2, U2.VSS; no longer D1.A, D2.A, J1G$1.GND, J1G$1.GND1, J1G$1.GND2, J1G$1.GND3, P1.GND, P2.2, R2.1, R5.1, R8.1, U1.1/GND, U1.103/GND, U1.104/GND, U1.109/GND, U1.110/GND, U1.115/GND, U1.116/GND, U1.121/GND, U1.13/GND, U1.133/GND, U1.134/GND, U1.139/GND, U1.14/NC, U1.140/GND, U1.145/GND, U1.146/GND, U1.151/GND, U1.152/GND, U1.163/GND, U1.164/GND, U1.169/GND, U1.170/GND, U1.181/GND, U1.182/GND, U1.187/GND, U1.188/GND, U1.19/GND, U1.195/GND, U1.196/GND, U1.20/NC, U1.25/GND, U1.26/GND, U1.31/GND, U1.32/GND, U1.37/GND, U1.38/GND, U1.43/GND, U1.44/GND, U1.49/GND, U1.50/GND, U1.55/GND, U1.56/GND, U1.61/GND, U1.62/GND, U1.67/GND, U1.68/GND, U1.7/GND, U1.73/GND, U1.74/GND, U1.79/GND, U1.8/NC, U1.80/GND, U1.85/GND, U1.86/GND, U1.91/GND, U1.92/GND, U1.97/GND, U1.98/GND, U2.GND, U4.VSS, U5.GND
- net N$1: now also PCB1.84/GPIO45, R13.2; no longer R10.2, U1.84/GPIO45
- net N$10: now also C7.1, R5.1, R7.2, U1.FB2; no longer R1.2, R2.2, U2.FB
- net N$11: now also L1.1, U1.LX1; no longer D2.C, L2.1, U3.SW
- net N$12: now also L2.1, U1.LX2; no longer D1.C, L1.1, U2.SW
- net N$14: now also R2.1; no longer R14.1
- net N$15: now also R19.2, U3.SCLK; no longer R15.2, U5.SCLK
- net N$16: now also R18.2, U3.MOSI; no longer R16.2, U5.MOSI
- net N$17: now also U3.*GPIO10; no longer U5.*GPIO10
- net N$18: now also R16.2, U3.*GPIO9; no longer R18.2, U5.*GPIO9
- net N$19: now also R15.2, U3.MISO; no longer R19.2, U5.MISO
- net N$2: now also C8.2, U1.EN2; no longer U3.EN
- net N$20: now also R14.2, U3.CS0; no longer R20.2, U5.CS0
- net N$3: now also LED2.C, U2.STAT; no longer CHARGE.C, U4.STAT
- net N$4: now also R9.2, U2.PROG; no longer R12.2, U4.PROG
- net N$5: now also LED2.A, R8.1; no longer CHARGE.A, R11.1
- net N$6: now also PCB1.28/GPIO28, R10.2; no longer R7.2, U1.28/GPIO28
- net N$7: now also PCB1.30/GPIO29, R11.2; no longer R8.2, U1.30/GPIO29
- net N$8: now also C5.1, R4.2, U1.FB1; no longer U2.EN
- net N$9: now also PCB1.82/GPIO44, R12.2; no longer R9.2, U1.82/GPIO44
- net SDIO_CLK: now also PCB1.75/GPIO22, R19.1; no longer R15.1, U1.75/GPIO22
- net SDIO_CMD: now also PCB1.77/GPIO23, R14.1; no longer R20.1, U1.77/GPIO23
- net SDIO_D0: now also PCB1.81/GPIO24, R15.1; no longer R19.1, U1.81/GPIO24
- net SDIO_D1: now also PCB1.83/GPIO25, R18.1; no longer R16.1, U1.83/GPIO25
- net SDIO_D2: now also PCB1.87/GPIO26, R16.1; no longer R18.1, U1.87/GPIO26
- net SDIO_D3: now also PCB1.89/GPIO27; no longer U1.89/GPIO27
- net SDIO_ID: now also PCB1.3/GPIO0, U3.CH_PD; no longer U1.3/GPIO0, U5.CH_PD
- net SDX_CLK: now also P2.CLK, PCB1.10/NC; no longer P1.CLK, U1.10/NC
- net SDX_CMD: now also P2.CMD, PCB1.12/NC; no longer P1.CMD, U1.12/NC
- net SDX_D0: now also P2.DAT0, PCB1.16/NC; no longer P1.DAT0, U1.16/NC
- net SDX_D1: now also P2.DAT1, PCB1.18/NC; no longer P1.DAT1, U1.18/NC
- net SDX_D2: now also P2.DAT2, PCB1.22/NC; no longer P1.DAT2, U1.22/NC
- net SDX_D3: now also P2.DAT3, PCB1.24/NC; no longer P1.DAT3, U1.24/NC
- net USB_N: now also PCB1.167/USB_DM**; no longer U1.167/USB_DM**
- net USB_P: now also PCB1.165/USB_DP**; no longer U1.165/USB_DP**
Other:
- moved on the sheet: C1, C2, C3, C4, D1, L1, L2, R1, R10, R11, R12, R13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
